Commit message: successful tested on isrl_fwmax robot

File: isrl_robot_description/urdf/robot1.xacro (robot description, xacro)
@@ -1,5 +1,5 @@
 <?xml version="1.0"?>
 <robot xmlns:xacro="http://ros.org/wiki/xacro" name="description" >
-  <link name="mobile_base_link">
+  <link name="base_link">
     <visual>
       <origin rpy="0 0 0" xyz="0 0 0" />

Commit message: add footprint, slamtoolbox package, navigation package

File: isrl_robot_description/urdf/robot1.xacro (robot description, xacro)
@@ -1,4 +1,12 @@
 <?xml version="1.0"?>
 <robot xmlns:xacro="http://ros.org/wiki/xacro" name="description" >
+<!--
+  <link name="base_footprint">
+  </link>
+  <joint name="base_to_footprint" type="fixed">
+    <parent link="base_footprint"/>
+    <child link="mobile_base_link"/>
+    <origin xyz="0.0 0.0 0.388" rpy="0.0 0.0 0.0"/>
+  </joint> -->
   <link name="base_link">
     <visual>
